File: hardware/electronics/deepreal-main-pcba/deepreal-main-pcba-visual.kicad_pcb (KiCad board)
At the start: 10 copper layers, 90 x 28 mm, 238 parts, among them J1 CX90M3-24P | BASELINE, J2 FH26W-51S-0.3SHW(97) | FLEX_S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, J3 FH26W-51S-0.3SHW(97) | FLEX_S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, J4 6-position low-profile | RESE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, J5 6-position low-profile | RESE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, U1 MIMX9596CVTXNAC | PINMAP_REQU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, U10 TPS259472LRPWR | BASELINE, U11 CYPD3177-24LQXQ | BASELINE, U12 HD3SS3212IRKSR | BASELINE, U13 DRV8213RTER | BASELINE, U14 DRV8213RTER | BASELINE, U15 MTFC32GBCAQTC-AAT | PINMAP_RE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, U16 AT24C64D-MAHM-T | BASELINE, U17 LMK1C1104DQFR | BASELINE, U18 AS5600L-AWLM | SUPPLY_RECHECK, U19 AS5600L-AWLM | SUPPLY_RECHECK, U2 LIFCL-17 | COMPILE_REQUIRED, U20 TMP117AIDRVR | BASELINE, U21 HEAD FACE SWITCH / TBD, U22 HEAD INTERACTION SWITCH / TBD, U3 LIFCL-17 | COMPILE_REQUIRED, U4 MT53E1G32D2FW-046 AAT:B | DDR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, U5 MPF0900AVNA2ES | SEQUENCE_REV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, U6 MPF5302BVNAAEP | SEQUENCE_REV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, U7 MPF5301BVNABEP | SEQUENCE_REV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, U8 TPS56637RPAR | CALC_REQUIRED, U9 TPS56637RPAR | CALC_REQUIRED

Commit message: fix(hardware): reroute visual copper around components
Parts:
- moved C80 79.3 mm to (27.5, 43.4)
- moved R19 79.3 mm to (105.5, 30.4)
- moved C112 75.4 mm to (105.5, 27.8)
- moved R17 75.4 mm to (102.9, 29.1)
- moved C107 71.5 mm to (100.3, 25.2)
- moved C58 71.5 mm to (28.8, 38.2)
- moved R21 71.5 mm to (96.4, 31.7)
- moved R6 71.5 mm to (101.6, 22.6)
- moved R8 71.5 mm to (96.4, 23.9)
- moved C73 67.6 mm to (28.8, 42.1)
- moved C12 67.6 mm to (100.3, 21.3)
- moved C88 67.6 mm to (26.2, 44.7)
- moved R15 67.6 mm to (104.2, 27.8)
- moved C27 63.7 mm to (106.8, 26.5)
- moved C61 59.8 mm to (23.6, 39.5)
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Routing:
- net (no net): vias 91 -> 113

Commit message: feat(hardware): establish gated PCBA engineering rebuild
Other:
- board text added: "SUPERSEDED CONCEPT - PUBLICATION PAUSED"
- board text removed: "PRODUCTION-INTENT VISUALIZATION"
Changed lines of the file:
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@@
 	(paper "A4")
 	(title_block
-		(title "DeepReal Main PCBA — PRODUCTION-INTENT VISUALIZATION")
+		(title "DeepReal Main PCBA — SUPERSEDED CONCEPT")
 		(rev "0.3-visual")
 		(company "DeepReal")
 		(comment 1 "90 x 28 mm; illustrative surface copper")
 		(comment 2 "NOT ELECTRICALLY ROUTED / NOT FOR FABRICATION")
-		(comment 3 "Website and investor presentation artifact only")
+		(comment 3 "PUBLICATION PAUSED - HISTORICAL ARTIFACT ONLY")
 	)
 	(layers
@@
 		(layer "Edge.Cuts")
 	)
-	(gr_text "PRODUCTION-INTENT VISUALIZATION"
+	(gr_text "SUPERSEDED CONCEPT - PUBLICATION PAUSED"
 		(at 65 46.6 0)
 		(layer "F.SilkS")
